Commit message: Added exported model from SW

File: src/capra_simulation/models/vincent.urdf (robot description, URDF)
Before this commit: robot capra6, 5 links, 4 joints
Links:
- link base_link: geometry collision mesh filename=package://capra_simulation/models/vincent/vincent.dae; visual mesh filename=package://capra_simulation/models/vincent/vincent.dae
