Commit message: itegrated navigation stack with the up to date urdf

File: src/robotcapra/urdf/robotcapra.urdf (robot description, URDF)
Before this commit: robot robotcapra, 1 links, 0 joints
Links:
- removed link robotcapra
- added link base_link, mass 23.124; collision mesh filename=package://robotcapra/meshes/robotcapra.STL; visual mesh filename=package://robotcapra/meshes/robotcapra.STL
- added link laser, mass 0; collision sphere radius=0.1
Joints:
- added joint joint1: type fixed, parent base_link, child laser, origin xyz=0.1 0.25 0.05 rpy=0 0 1.5707963267949

Commit message: Added sdf to urdf converter and modified robot model

File: src/robotcapra/urdf/robotcapra.urdf (robot description, URDF)
Before this commit: robot robotcapra, 2 links, 1 joints
Links:
- removed link base_link
- added link capra6__base_link, mass 23.124; collision mesh filename=package://robotcapra/meshes/robotcapra.stl scale=1 1 1; collision sphere radius=0.1
- added link capra6__link_0, mass 1; collision cylinder length=0.1 radius=0.05; visual cylinder length=0.1 radius=0.05
- added link capra6__link_0_clone, mass 1; collision cylinder length=0.1 radius=0.05; visual cylinder length=0.1 radius=0.05
- added link capra6__link_0_clone_0, mass 1; collision cylinder length=0.1 radius=0.05; visual cylinder length=0.1 radius=0.05
- added link capra6__link_0_clone_1, mass 1; collision cylinder length=0.1 radius=0.05; visual cylinder length=0.1 radius=0.05
Joints:
- added joint capra6__JOINT_WHEEL_F_L: type revolute, parent capra6__base_link, child capra6__link_0_clone, origin xyz=-0.05127  0.15058 -0.19177 rpy=0  0  0, axis 1  0  0, limit lower=-1.79769e+308 upper=1.79769e+308 effort=-1.0 velocity=-1.0
- added joint capra6__JOINT_WHEEL_F_R: type revolute, parent capra6__base_link, child capra6__link_0, origin xyz=0.28816  0.15376 -0.19177 rpy=0  0  0, axis -1  0  0, limit lower=-1.79769e+308 upper=1.79769e+308 effort=-1.0 velocity=-1.0
- added joint capra6__JOINT_WHEEL_R_L: type revolute, parent capra6__base_link, child capra6__link_0_clone_1, origin xyz=-0.05803 -0.15462 -0.19177 rpy=0  0  0, axis 1  0  0, limit lower=-1.79769e+308 upper=1.79769e+308 effort=-1.0 velocity=-1.0
- added joint capra6__JOINT_WHEEL_R_R: type revolute, parent capra6__base_link, child capra6__link_0_clone_0, origin xyz=0.29719 -0.15535 -0.19177 rpy=0  0  0, axis -1  0  0, limit lower=-1.79769e+308 upper=1.79769e+308 effort=-1.0 velocity=-1.0
- joint joint1: parent base_link -> capra6__base_link

Commit message: Starting cleanup of Simulation launch file

File: src/robotcapra/urdf/robotcapra.urdf (robot description, URDF)
Before this commit: robot capra6, 6 links, 5 joints
Links:
- removed link capra6__base_link
- added link base_link, mass 23.124; collision mesh filename=package://robotcapra/meshes/robotcapra.stl scale=1 1 1; collision sphere radius=0.1
Joints:
- joint capra6__JOINT_WHEEL_F_L: parent capra6__base_link -> base_link
- joint capra6__JOINT_WHEEL_F_R: parent capra6__base_link -> base_link
- joint capra6__JOINT_WHEEL_R_L: parent capra6__base_link -> base_link
- joint capra6__JOINT_WHEEL_R_R: parent capra6__base_link -> base_link
- joint joint1: parent capra6__base_link -> base_link
