Commit message: Add fixed joint from laser_tower to laser

File: src/capra_simulation/models/urdf/capra_robot.urdf (robot description, URDF)
Before this commit: robot capra_robot, 6 links, 5 joints
Links:
- added link capra_robot__laser_tower, mass 1.0; collision box size=.01 .01 .1; visual box size=.01 .01 .1
- link base_link: mass 0 -> 23.124
- link capra_robot__laser: mass 0 -> .1; geometry collision box size=.01 .01 .01; visual box size=.01 .01 .01
- link capra_robot__left_wheel_back: mass 0 -> 1.0
- link capra_robot__left_wheel_front: mass 0 -> 1.0
- link capra_robot__right_wheel_back: mass 0 -> 1.0
- link capra_robot__right_wheel_front: mass 0 -> 1.0
Joints:
- removed joint capra_robot__laser_tower
- added joint capra_robot__laser_joint: type fixed, parent capra_robot__laser_tower, child capra_robot__laser, origin xyz=0  0  0.05 rpy=0  0  0, axis 0  0  1, limit lower=0 upper=0 effort=0 velocity=0
- added joint capra_robot__laser_tower_joint: type fixed, parent base_link, child capra_robot__laser_tower, origin xyz=0.195  0     0.16 rpy=0  0  0, axis 0  0  1, limit lower=0 upper=0 effort=0 velocity=0
- joint capra_robot__left_wheel_back_hinge: limit lower=0 upper=0 effort=0 velocity=0 -> lower=-1.79769e+308 upper=1.79769e+308 effort=-1.0 velocity=-1.0
- joint capra_robot__left_wheel_front_hinge: limit lower=0 upper=0 effort=0 velocity=0 -> lower=-1.79769e+308 upper=1.79769e+308 effort=-1.0 velocity=-1.0
- joint capra_robot__right_wheel_back_hinge: limit lower=0 upper=0 effort=0 velocity=0 -> lower=-1.79769e+308 upper=1.79769e+308 effort=-1.0 velocity=-1.0
- joint capra_robot__right_wheel_front_hinge: limit lower=0 upper=0 effort=0 velocity=0 -> lower=-1.79769e+308 upper=1.79769e+308 effort=-1.0 velocity=-1.0

Commit message: Fix rotation axis to z axis for wheel joints

File: src/capra_simulation/models/urdf/capra_robot.urdf (robot description, URDF)
Before this commit: robot capra_robot, 7 links, 6 joints
Links:
- link base_link: geometry collision box size=.4 .2 .1; visual box size=.4 .2 .1
Joints:
- joint capra_robot__left_wheel_back_hinge: axis 0  1  0 -> 0  0  1
- joint capra_robot__left_wheel_front_hinge: axis 0  1  0 -> 0  0  1
- joint capra_robot__right_wheel_back_hinge: axis 0  1  0 -> 0  0  1
- joint capra_robot__right_wheel_front_hinge: axis 0  1  0 -> 0  0  1

Commit message: Add camera to capra_robot on sensor tower

File: src/capra_simulation/models/urdf/capra_robot.urdf (robot description, URDF)
Before this commit: robot capra_robot, 7 links, 6 joints
Links:
- removed link capra_robot__laser_tower
- added link capra_robot__camera, mass .1; collision box size=.01 .01 .01; visual box size=.01 .01 .01
- added link capra_robot__sensor_tower, mass 1.0; collision box size=.01 .01 .1; visual box size=.01 .01 .1
Joints:
- removed joint capra_robot__laser_tower_joint
- added joint capra_robot__camera_joint: type fixed, parent capra_robot__sensor_tower, child capra_robot__camera, origin xyz=0  0  0.05 rpy=0  0  0, axis 0  0  1, limit lower=0 upper=0 effort=0 velocity=0
- added joint capra_robot__sensor_tower_joint: type fixed, parent base_link, child capra_robot__sensor_tower, origin xyz=0.195  0     0.16 rpy=0  0  0, axis 0  0  1, limit lower=0 upper=0 effort=0 velocity=0
- joint capra_robot__laser_joint: parent capra_robot__laser_tower -> capra_robot__sensor_tower

Commit message: Add IMU sensor centered on top of base link

File: src/capra_simulation/models/urdf/capra_robot.urdf (robot description, URDF)
Before this commit: robot capra_robot, 8 links, 7 joints
Links:
- added link capra_robot__IMU, mass .1; collision box size=.01 .01 .05; visual box size=.01 .01 .05
Joints:
- added joint capra_robot__IMU_joint: type fixed, parent base_link, child capra_robot__IMU, origin xyz=0  0  0.135 rpy=0  0  0, axis 0  0  1, limit lower=0 upper=0 effort=0 velocity=0
